File: A5256.kicad_pcb (KiCad board)
At the start: 6 copper layers, 127.7 x 49.1 mm, 315 parts, among them IC1 LTM8074EY#PBF, IC2 LT3581IDE#PBF, IC3 LTM8074EY#PBF, IC4 LT3015IMSE-15#PBF, IC5 LT1963AES8-3.3#TRPBF, IC6 AD5673RBCPZ-1, J1 5-1775444-3, J2 09185346323, J3 EPL.00.250.NTN, J4 09195346829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

Commit message: quasi terminato il back
Parts:
- moved R5 2.77 mm to (201.4, 90.7), turned to 90 degrees
- moved R2 1.13 mm to (142.7, 89.5)
- moved R1 1.13 mm to (141.2, 89.5)
- moved R7 0.35 mm to (188.8, 90.8)
- moved C8 0.34 mm to (188.7, 89.3)
- turned C1 to 0 degrees
- turned L1 to 0 degrees
Routing:
- net /Power Supply/-5V: track 20.9 -> 32.7 mm
- net +12V: track 6.28 -> 14.1 mm
- net Net-(IC2-SS): track 0.00 -> 1.92 mm
- net Net-(IC2-~{FAULT}): track 6.24 -> 7.86 mm
- net Net-(IC2-RT): track 0.00 -> 1.58 mm
- net /VOUT13: track 50.5 -> 51.9 mm
- net /CH0/SCL: track 54.3 -> 55.5 mm
- net /CH0/SDA: track 59.8 -> 60.9 mm
- net 4V5: track 89.5 -> 90.5 mm
- net GND: vias 204 -> 216

Commit message: fatto piano di power
Parts:
- added NT1: NetTie_4, NetTie:NetTie-4_SMD_Pad0.5mm, F.Cu at (193.8, 89.6)
- moved C1 4.50 mm to (181.7, 88.9)
- moved R4 4.21 mm to (194.8, 83.0)
- moved IC2 3.42 mm to (193.0, 87.8)
- moved C9 3.10 mm to (200.3, 83.1), turned to 180 degrees
- moved R7 3.08 mm to (188.6, 87.7)
- moved C8 3.05 mm to (188.5, 86.2)
- moved R8 2.37 mm to (198.1, 86.5)
- moved C7 2.36 mm to (196.2, 86.5)
- moved R5 1.37 mm to (201.1, 89.4)
- moved C67 0.53 mm to (180.5, 99.9)
- moved C69 0.28 mm to (176.0, 109.6)
Connections:
- C1 pad 2: GND -> /Power Supply/GND_out
- C2 pad 2: GND -> /Power Supply/GND_in
- D1 pad 1: GND -> /Power Supply/GND_diode
- J4 pad 33: unconnected-(J4-Pad33) -> GND
- J4 pad 34: unconnected-(J4-Pad34) -> GND
Routing:
- net +12V: track 14.1 -> 137.0 mm
- net /Vb2: track 105.6 -> 27.9 mm
- net Net-(C9-Pad1): track 1.76 -> 8.32 mm
- net 4V5: track 90.5 -> 94.4 mm, vias 42 -> 44
- net /Signals 9-10/INB+: track 49.2 -> 46.3 mm
- net Net-(JP29-C): track 47.6 -> 44.9 mm
- net Net-(U1-VOUTA): track 40.0 -> 42.0 mm
- net Net-(JP14-C): track 45.6 -> 43.9 mm
- net Net-(JP26-C): track 58.1 -> 56.5 mm
- net /Signals 11-12/INB+: track 69.3 -> 67.7 mm
- net Net-(U1-VOUTB): track 53.8 -> 55.4 mm
- net -4V5: track 146.2 -> 147.7 mm
- net /Signals 9-10/INA+: track 56.8 -> 55.3 mm
- net Net-(JP34-C): track 67.9 -> 66.4 mm
- net /Signals 3-4/INB+: track 46.5 -> 45.1 mm
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- added copper zone on In4.Cu, net +1V7
- added copper zone on In4.Cu, net -4V5
- added copper zone on B.Cu, net /Power Supply/GND_diode
- added copper zone on F.Cu, net /Power Supply/GND_diode
- added copper zone on B.Cu, net /Power Supply/GND_in
- added copper zone on F.Cu, net /Power Supply/GND_in
- added copper zone on B.Cu, net /Power Supply/GND_out
- added copper zone on F.Cu, net /Power Supply/GND_out
- added copper zone on In4.Cu, net 4V5
- added copper zone on F.Cu, net GND
