File: A5256.kicad_sch (KiCad schematic)
At the start: 9 parts, among them J1 5-1775444-3, J2 09185346323, J3 EPL.00.250.NTN, J4 09195346829, J6 5-1775444-3

Commit message: fatto piano di power
Connections:
- net GND: now also J4.33, J4.34
- no-connect marks 6 -> 4
Changed lines of the file:
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@@
 		(color 0 0 0 0)
 	)
-	(no_connect
-		(at 519.43 237.49)
-	)
-	(no_connect
-		(at 542.29 237.49)
+	(junction
+		(at 532.13 242.57)
+		(diameter 0)
+		(color 0 0 0 0)
 	)
 	(no_connect
@@
 	(wire
 		(pts
+			(xy 516.89 242.57) (xy 532.13 242.57)
+		)
+		(stroke
+			(width 0)
+			(type default)
+		)
+	)
+	(wire
+		(pts
 			(xy 312.42 160.02) (xy 322.58 160.02)
 		)
@@
 	(wire
 		(pts
+			(xy 532.13 242.57) (xy 532.13 245.11)
+		)
+		(stroke
+			(width 0)
+			(type default)
+		)
+	)
+	(wire
+		(pts
 			(xy 66.04 214.63) (xy 66.04 217.17)
 		)
@@
 	(wire
 		(pts
+			(xy 532.13 242.57) (xy 546.1 242.57)
+		)
+		(stroke
+			(width 0)
+			(type default)
+		)
+	)
+	(wire
+		(pts
 			(xy 542.29 229.87) (xy 549.91 229.87)
 		)
@@
 	(wire
 		(pts
+			(xy 519.43 237.49) (xy 516.89 237.49)
+		)
+		(stroke
+			(width 0)
+			(type default)
+		)
+	)
+	(wire
+		(pts
 			(xy 66.04 199.39) (xy 64.77 199.39)
 		)
@@
 	(wire
 		(pts
+			(xy 546.1 242.57) (xy 546.1 237.49)
+		)
+		(stroke
+			(width 0)
+			(type default)
+		)
+	)
+	(wire
+		(pts
 			(xy 63.5 165.1) (xy 63.5 167.64)
 		)
@@
 	(wire
 		(pts
+			(xy 546.1 237.49) (xy 542.29 237.49)
+		)
+		(stroke
+			(width 0)
+			(type default)
+		)
+	)
+	(wire
+		(pts
 			(xy 60.96 68.58) (xy 60.96 72.39)
 		)
@@
 	(wire
 		(pts
+			(xy 516.89 237.49) (xy 516.89 242.57)
+		)
+		(stroke
+			(width 0)
+			(type default)
+		)
+	)
+	(wire
+		(pts
 			(xy 322.58 245.11) (xy 311.15 245.11)
 		)
@@
 					(unit 1)
 				)
+			)
+		)
+	)
+	(symbol
+		(lib_id "power:GND")
+		(at 532.13 245.11 0)
+		(unit 1)
+		(exclude_from_sim no)
+		(in_bom yes)
+		(on_board yes)
+		(dnp no)
+		(property "Reference" "#PWR0210"
+			(at 532.13 251.46 0)
+			(effects
+				(font
+					(size 1.27 1.27)
+				)
+				(hide yes)
+			)
+		)
+		(property "Value" "GND"
+			(at 532.13 248.666 0)
+			(effects
+				(font
+					(size 1.27 1.27)
+				)
+			)
+		)
+		(property "Footprint" ""
+			(at 532.13 245.11 0)
+			(effects
+				(font
+					(size 1.27 1.27)
+				)
+				(hide yes)
+			)
+		)
+		(property "Datasheet" ""
+			(at 532.13 245.11 0)
+			(effects
+				(font
+					(size 1.27 1.27)
+				)
+				(hide yes)
+			)
+		)
+		(property "Description" "Power symbol creates a global label with name \"GND\" , ground"
+			(at 532.13 245.11 0)
+			(effects
+				(font
+					(size 1.27 1.27)
+				)
+				(hide yes)
+			)
+		)
+		(pin "1"
+		)
+		(instances
+			(project "A5256"
+				(path "/59e0b50f-8080-4ed9-9b83-2233f3b14569"
+					(reference "#PWR0210")
+					(unit 1)
+				)
