File: Signals 11-12.kicad_sch (KiCad schematic)
At the start: 32 parts, among them U15 LMH7322, U16 AD8657

Commit message: modificato pad esposti
Connections:
- net -4V5: now also U15.25 (EP)
- net GND: no longer U15.25 (EP)
Changed lines of the file:
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@@
 	(wire
 		(pts
+			(xy 170.18 209.55) (xy 170.18 213.36)
+		)
+		(stroke
+			(width 0)
+			(type default)
+		)
+	)
+	(wire
+		(pts
 			(xy 210.82 222.25) (xy 210.82 224.79)
 		)
@@
 	(wire
 		(pts
+			(xy 170.18 213.36) (xy 162.56 213.36)
+		)
+		(stroke
+			(width 0)
+			(type default)
+		)
+	)
+	(wire
+		(pts
 			(xy 153.67 182.88) (xy 157.48 182.88)
 		)
@@
 	(wire
 		(pts
-			(xy 246.38 60.96) (xy 251.46 60.96)
+			(xy 162.56 210.82) (xy 162.56 213.36)
 		)
 		(stroke
@@
 	(wire
 		(pts
-			(xy 224.79 54.61) (xy 223.52 54.61)
+			(xy 246.38 60.96) (xy 251.46 60.96)
 		)
 		(stroke
@@
 	(wire
 		(pts
-			(xy 214.63 101.6) (xy 214.63 109.22)
+			(xy 224.79 54.61) (xy 223.52 54.61)
 		)
 		(stroke
@@
 	(wire
 		(pts
-			(xy 267.97 52.07) (xy 252.73 52.07)
+			(xy 214.63 101.6) (xy 214.63 109.22)
 		)
 		(stroke
@@
 	(wire
 		(pts
-			(xy 170.18 209.55) (xy 170.18 213.36)
+			(xy 267.97 52.07) (xy 252.73 52.07)
 		)
 		(stroke
@@
 	)
 	(symbol
-		(lib_id "power:GND")
-		(at 170.18 213.36 0)
-		(mirror y)
-		(unit 1)
-		(exclude_from_sim no)
-		(in_bom yes)
-		(on_board yes)
-		(dnp no)
-		(property "Reference" "#PWR0171"
-			(at 170.18 219.71 0)
-			(effects
-				(font
-					(size 1.27 1.27)
-				)
-				(hide yes)
-			)
-		)
-		(property "Value" "GND"
-			(at 167.386 213.36 0)
-			(effects
-				(font
-					(size 1.27 1.27)
-				)
-			)
-		)
-		(property "Footprint" ""
-			(at 170.18 213.36 0)
-			(effects
-				(font
-					(size 1.27 1.27)
-				)
-				(hide yes)
-			)
-		)
-		(property "Datasheet" ""
-			(at 170.18 213.36 0)
-			(effects
-				(font
-					(size 1.27 1.27)
-				)
-				(hide yes)
-			)
-		)
-		(property "Description" "Power symbol creates a global label with name \"GND\" , ground"
-			(at 170.18 213.36 0)
-			(effects
-				(font
-					(size 1.27 1.27)
-				)
-				(hide yes)
-			)
-		)
-		(pin "1"
-		)
-		(instances
-			(project "A5256"
-				(path "/59e0b50f-8080-4ed9-9b83-2233f3b14569/fb2a3acf-1eac-44eb-9b9f-bd44f7e9ca71"
-					(reference "#PWR0171")
-					(unit 1)
-				)
-			)
-		)
-	)
-	(symbol
 		(lib_id "Device:R")
 		(at 176.53 228.6 0)
@@
 					(unit 1)
 				)
+			)
+		)
+	)
+	(symbol
+		(lib_id "power:-8V")
+		(at 162.56 210.82 0)
+		(mirror y)
+		(unit 1)
+		(exclude_from_sim no)
+		(in_bom yes)
+		(on_board yes)
+		(dnp no)
+		(property "Reference" "#PWR0151"
+			(at 162.56 214.63 0)
+			(effects
+				(font
+					(size 1.27 1.27)
+				)
+				(hide yes)
+			)
+		)
+		(property "Value" "-4V5"
+			(at 162.814 207.01 0)
+			(effects
+				(font
+					(size 1.27 1.27)
+				)
+			)
+		)
+		(property "Footprint" ""
+			(at 162.56 210.82 0)
+			(effects
+				(font
+					(size 1.27 1.27)
+				)
+				(hide yes)
+			)
+		)
+		(property "Datasheet" ""
+			(at 162.56 210.82 0)
+			(effects
+				(font
+					(size 1.27 1.27)
+				)
+				(hide yes)
+			)
+		)
+		(property "Description" "Power symbol creates a global label with name \"-8V\""
+			(at 162.56 210.82 0)
+			(effects
+				(font
+					(size 1.27 1.27)
+				)
+				(hide yes)
+			)
+		)
+		(pin "1"
+		)
+		(instances
+			(project "A5256"
+				(path "/59e0b50f-8080-4ed9-9b83-2233f3b14569/fb2a3acf-1eac-44eb-9b9f-bd44f7e9ca71"
+					(reference "#PWR0151")
+					(unit 1)
+				)
