File: Signals 7-8.kicad_sch (KiCad schematic)
At the start: 32 parts, among them U11 LMH7322, U12 AD8657

Commit message: modificato pad esposti
Connections:
- net -4V5: now also U11.25 (EP)
- net GND: no longer U11.25 (EP)
Changed lines of the file:
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@@
 	(wire
 		(pts
+			(xy 168.91 213.36) (xy 161.29 213.36)
+		)
+		(stroke
+			(width 0)
+			(type default)
+		)
+	)
+	(wire
+		(pts
 			(xy 152.4 198.12) (xy 144.78 198.12)
 		)
@@
 	(wire
 		(pts
+			(xy 168.91 209.55) (xy 168.91 213.36)
+		)
+		(stroke
+			(width 0)
+			(type default)
+		)
+	)
+	(wire
+		(pts
 			(xy 144.78 58.42) (xy 144.78 54.61)
 		)
@@
 	(wire
 		(pts
+			(xy 161.29 210.82) (xy 161.29 213.36)
+		)
+		(stroke
+			(width 0)
+			(type default)
+		)
+	)
+	(wire
+		(pts
 			(xy 134.62 54.61) (xy 144.78 54.61)
 		)
@@
 	(wire
 		(pts
-			(xy 168.91 209.55) (xy 168.91 213.36)
-		)
-		(stroke
-			(width 0)
-			(type default)
-		)
-	)
-	(wire
-		(pts
 			(xy 166.37 85.09) (xy 166.37 88.9)
 		)
@@
 	)
 	(symbol
-		(lib_id "power:GND")
-		(at 168.91 213.36 0)
+		(lib_id "power:-8V")
+		(at 161.29 210.82 0)
 		(mirror y)
 		(unit 1)
@@
 		(on_board yes)
 		(dnp no)
-		(property "Reference" "#PWR0131"
-			(at 168.91 219.71 0)
+		(property "Reference" "#PWR0111"
+			(at 161.29 214.63 0)
 			(effects
 				(font
@@
 			)
 		)
-		(property "Value" "GND"
-			(at 166.116 213.36 0)
+		(property "Value" "-4V5"
+			(at 161.544 207.01 0)
 			(effects
 				(font
@@
 		)
 		(property "Footprint" ""
-			(at 168.91 213.36 0)
+			(at 161.29 210.82 0)
 			(effects
 				(font
@@
 		)
 		(property "Datasheet" ""
-			(at 168.91 213.36 0)
+			(at 161.29 210.82 0)
 			(effects
 				(font
@@
 			)
 		)
-		(property "Description" "Power symbol creates a global label with name \"GND\" , ground"
-			(at 168.91 213.36 0)
+		(property "Description" "Power symbol creates a global label with name \"-8V\""
+			(at 161.29 210.82 0)
 			(effects
 				(font
@@
 			(project "A5256"
 				(path "/59e0b50f-8080-4ed9-9b83-2233f3b14569/3c9e057b-9a4b-4b52-bf18-cca9fbecbed2"
-					(reference "#PWR0131")
+					(reference "#PWR0111")
 					(unit 1)
 				)
