File: Trigger 0.kicad_sch (KiCad schematic)
At the start: 46 parts, among them IC6 AD5673RBCPZ-1, U1 LTC2627IDE-1_PBF, U2 AD8657, U3 AD8657, U4 LMH7322

Commit message: posizionato riferimenti in modo corretto
Parts:
- TP1: value TestPoint IN 0A -> TestPoint IN 0B
- TP2: value TestPoint IN 0B -> TestPoint IN 0A
Changed lines of the file:
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@@
 			)
 		)
-		(property "Value" "TestPoint IN 0B"
+		(property "Value" "TestPoint IN 0A"
 			(at 372.364 173.99 90)
 			(effects
@@
 			)
 		)
-		(property "Value" "TestPoint IN 0A"
+		(property "Value" "TestPoint IN 0B"
 			(at 372.364 147.32 90)
 			(effects

Commit message: modificato pad esposti
Connections:
- net -4V5: now also U4.25 (EP)
- net GND: no longer U4.25 (EP)
Changed lines of the file:
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@@
 	)
 	(junction
-		(at 231.14 195.58)
-		(diameter 0)
-		(color 0 0 0 0)
-	)
-	(junction
 		(at 166.37 82.55)
 		(diameter 0)
@@
 	(wire
 		(pts
-			(xy 234.95 195.58) (xy 231.14 195.58)
+			(xy 179.07 170.18) (xy 185.42 170.18)
 		)
 		(stroke
@@
 	(wire
 		(pts
-			(xy 179.07 170.18) (xy 185.42 170.18)
+			(xy 234.95 195.58) (xy 237.49 195.58)
 		)
 		(stroke
@@
 	(wire
 		(pts
+			(xy 237.49 194.31) (xy 237.49 195.58)
+		)
+		(stroke
+			(width 0)
+			(type default)
+		)
+	)
+	(wire
+		(pts
 			(xy 231.14 187.96) (xy 231.14 195.58)
 		)
@@
 					(unit 1)
 				)
+			)
+		)
+	)
+	(symbol
+		(lib_id "power:-8V")
+		(at 237.49 194.31 0)
+		(unit 1)
+		(exclude_from_sim no)
+		(in_bom yes)
+		(on_board yes)
+		(dnp no)
+		(fields_autoplaced yes)
+		(property "Reference" "#PWR012"
+			(at 237.49 198.12 0)
+			(effects
+				(font
+					(size 1.27 1.27)
+				)
+				(hide yes)
+			)
+		)
+		(property "Value" "-4V5"
+			(at 237.49 189.23 0)
+			(effects
+				(font
+					(size 1.27 1.27)
+				)
+			)
+		)
+		(property "Footprint" ""
+			(at 237.49 194.31 0)
+			(effects
+				(font
+					(size 1.27 1.27)
+				)
+				(hide yes)
+			)
+		)
+		(property "Datasheet" ""
+			(at 237.49 194.31 0)
+			(effects
+				(font
+					(size 1.27 1.27)
+				)
+				(hide yes)
+			)
+		)
+		(property "Description" "Power symbol creates a global label with name \"-8V\""
+			(at 237.49 194.31 0)
+			(effects
+				(font
+					(size 1.27 1.27)
+				)
+				(hide yes)
+			)
+		)
+		(pin "1"
+		)
+		(instances
+			(project "A5256"
+				(path "/59e0b50f-8080-4ed9-9b83-2233f3b14569/e43a2eda-b2d3-42a8-b923-dee4aca0821d"
+					(reference "#PWR012")
+					(unit 1)
+				)
